File: block diagram/block diagram.kicad_sch (KiCad schematic)
At the start: 0 parts

Commit message: add actual content
Parts:
- added SW?: SW_SP3T, symbol Switch:SW_SP3T
Other:
- added sheet AM reciever (am_receiver.kicad_sch)
- added sheet Bluetooth (bluetooth.kicad_sch)
- added sheet FM receiver (fm_receiver.kicad_sch)
- added sheet Power (power.kicad_sch)
