File: block diagram/untitled.kicad_sch (KiCad schematic)
At the start: 0 parts

Commit message: diagrammed bt chip, please fix formatting
Parts:
- added BT1: (no value), symbol son_kicad:bt_chip
- added C1: C, symbol Device:C
- added L1: 100 mH, symbol Device:L
- added R1: 51K, symbol Device:R
- added R13: 9.1K, symbol Device:R
- added R19: 0, symbol Device:R
- added R7: 33K, symbol Device:R
Connections:
- new net: C1.1, L1.1
- new net: R1.1, R13.1, R19.1, R7.1
- new net GND1: C1.2
- new net VCC 5V: L1.2
- new net bt on/off: R19.2
- new net next: R7.2
- new net pause: R1.2
- new net prev: R13.2
- no-connect marks 0 -> 2
Other:
- note added: "LINK TO PART"
- note added: "audio out"
- note added: "need to decide switching mechanism! and whether to integrate the on/off into main board! and whether all 4 pins are needed or if it's too much. because like technically you can skip tracks on your phone"
- note added: "power ground"
